Commit message: sensors added

File: description/robot.urdf.xacro (robot description, xacro)
@@ -3,3 +3,5 @@
     <xacro:include filename="robot_core.xacro" />
     <xacro:include filename="gazebo_control.xacro" />
+    <xacro:include filename="lidar.xacro" />
+    <xacro:include filename="camera.xacro" />
 </robot>

File: description/robot_core.xacro (robot description, xacro)
@@ -15,4 +15,7 @@
     <material name="blue">
         <color rgba="0.2 0.2 1 1"/>
+    </material>
+    <material name="red">
+        <color rgba="1 0.2 0.2 1"/>
     </material>
     <!--Chassis-->

Commit message: Depth Camera, Ros_Control, and Joy Stick Control

File: description/robot.urdf.xacro (robot description, xacro)
@@ -2,6 +2,8 @@
 <robot xmlns:xacro="http://www.ros.org/wiki/xacro"  name="robot">
     <xacro:include filename="robot_core.xacro" />
-    <xacro:include filename="gazebo_control.xacro" />
+    <!-- <xacro:include filename="gazebo_control.xacro" /> -->
+    <xacro:include filename="ros_control.xacro" />
     <xacro:include filename="lidar.xacro" />
-    <xacro:include filename="camera.xacro" />
+    <!-- <xacro:include filename="camera.xacro" /> -->
+    <xacro:include filename="depth_camera.xacro" />
 </robot>

File: description/robot_core.xacro (robot description, xacro)
@@ -53,4 +53,5 @@
         <child link="left_wheel"/>
         <axis xyz="0 0 1"/>
+        <limit effort="100" velocity="10" lower="-10" upper="10"/>
     </joint>
     <link name="left_wheel">
@@ -79,4 +80,5 @@
         <child link="right_wheel"/>
         <axis xyz="0 0 -1"/>
+        <limit effort="100" velocity="10" lower="-10" upper="10"/>
     </joint>
     <link name="right_wheel">
