Commit message: slam and navigation stack

File: description/robot_core.xacro (robot description, xacro)
@@ -21,6 +21,12 @@
     <!--Chassis-->
     <link name="base_link" />
+    <joint name="base_footprint_joint" type="fixed">
+        <origin xyz="0 0 0" rpy="0 0 0"/>
+        <parent link="base_link"/>
+        <child link="base_footprint"/>
+    </joint>
+    <link name="base_footprint" />
     <joint name = "chassis_joint" type="fixed">
-        <origin xyz="-0.1 0 0" rpy="0 0 0"/>
+        <origin xyz="0 0 0" rpy="0 0 0"/>
         <parent link="base_link"/>
         <child link="chassis"/>

Commit message: Wheels position corrected

File: description/robot_core.xacro (robot description, xacro)
@@ -22,5 +22,5 @@
     <link name="base_link" />
     <joint name="base_footprint_joint" type="fixed">
-        <origin xyz="0 0 0" rpy="0 0 0"/>
+        <origin xyz="0 0 -0.05" rpy="0 0 0"/>
         <parent link="base_link"/>
         <child link="base_footprint"/>
@@ -55,5 +55,5 @@
     <!--LEFT WHEEL-->
     <joint name = "left_wheel_joint" type="continuous">
-        <origin xyz="0 0.175 0" rpy="-${M_PI/2} 0 0"/>
+        <origin xyz="0.05 0.175 0" rpy="-${M_PI/2} 0 0"/>
         <parent link="base_link"/>
         <child link="left_wheel"/>
@@ -82,5 +82,5 @@
     <!--RIGHT WHEEL-->
     <joint name = "right_wheel_joint" type="continuous">
-        <origin xyz="0 -0.175 0" rpy="${M_PI/2} 0 0"/>
+        <origin xyz="0.05 -0.175 0" rpy="${M_PI/2} 0 0"/>
         <parent link="base_link"/>
         <child link="right_wheel"/>
